File: hardware/blüp/blüp.kicad_pcb (KiCad board)
At the start: 4 copper layers, 70 x 70 mm, 75 parts, among them J1 USB4105-GF-A, J2 Pump / JST XH, Q1 AO3401A, SW1 RESET, SW2 BOOT, U1 ESP32-S3-MINI-1-N8, U2 STUSB4500QTR, U3 AP63203WU, U4 AP63200WU-7, U5 TPS259620DDAR

Commit message: first cut CAD + PCB
Parts:
- moved SW2 50.0 mm to (113.0, 75.0)
- moved R13 18.0 mm to (115.0, 122.2)
- moved R12 14.9 mm to (115.0, 120.0)
- moved C17 12.4 mm to (125.5, 94.0), turned to 0 degrees
- moved C14 10.8 mm to (114.5, 97.2), turned to 0 degrees
- moved C10 10.2 mm to (158.0, 118.8)
- moved D5 10.2 mm to (158.0, 122.8)
- moved Q1 9.55 mm to (153.5, 119.0)
- moved C23 9.20 mm to (154.5, 89.5), turned to 90 degrees
- moved R7 9.03 mm to (149.2, 122.2)
- moved R8 9.03 mm to (149.2, 117.8)
- moved R9 9.03 mm to (149.2, 120.0)
- moved C15 8.34 mm to (114.5, 94.8), turned to 0 degrees
- moved C5 8.30 mm to (152.2, 114.4)
- moved C6 8.13 mm to (149.2, 115.5), turned to 0 degrees
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Routing:
- net +3V3: track 0.00 -> 143.0 mm, vias 0 -> 8
- net /VBUS_SW: track 0.00 -> 122.1 mm, vias 0 -> 17
- net GND: track 0.00 -> 84.7 mm, vias 0 -> 62
- net +12V: track 0.00 -> 75.5 mm, vias 0 -> 2
- net /VBUS: track 0.00 -> 74.1 mm
- net /REG12_EN: track 0.00 -> 64.3 mm, vias 0 -> 2
- net /PD_PDO2_N: track 0.00 -> 63.3 mm, vias 0 -> 3
- net /PD_ALERT: track 0.00 -> 58.1 mm, vias 0 -> 2
- net /PD_RESET: track 0.00 -> 50.2 mm, vias 0 -> 2
- net /PUMP_ILM: track 0.00 -> 46.6 mm, vias 0 -> 2
- net /PUMP_FLT_N: track 0.00 -> 46.5 mm, vias 0 -> 2
- net /I2C_SDA: track 0.00 -> 43.3 mm, vias 0 -> 4
- net /I2C_SCL: track 0.00 -> 41.1 mm, vias 0 -> 4
- net /PD_EN_SNK: track 0.00 -> 39.0 mm, vias 0 -> 3
- net /PUMP_EN: track 0.00 -> 33.4 mm, vias 0 -> 2
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- added copper zone on B.Cu, net GND
- added copper zone on F.Cu, net GND
- added copper zone on In1.Cu, net GND
- added copper zone on In2.Cu, net GND
